File: KiCad/ze-keyboard.kicad_pcb (KiCad board)
At the start: 2 copper layers, 211 parts, among them J1 Conn_01x05, J2 USB_C_Receptacle_USB2.0, SW1 Flash, SW2 Reset, SW3 RotaryEncoder_Switch, U1 XC6206PxxxMR, U2 RP2040, U3 W25Q128JVS, U4 SRV05-4, Y1 Crystal_GND24_Small

Commit message: fix flipped keyboard, and finish routing mcu
Parts:
- C1, C10, C11, C12, C13, C14, C15, C16, C2, C3, C4, C5, C6, C7, C8, C9, D1, D10, D11, D12, D13, D14, D15, D16, D17, D18, D19, D2, D20, D21, D22, D23, D24, D25, D26, D27, D28, D29, D3, D30, D31, D32, D33, D34, D35, D36, D37, D38, D39, D4, D40, D41, D42, D43, D44, D45, D46, D47, D48, D49, D5, D50, D51, D52, D53, D54, D55, D56, D57, D58, D59, D6, D60, D61, D62, D63, D64, D65, D66, D67, D68, D69, D7, D70, D71, D72, D73, D74, D75, D76, D77, D78, D79, D8, D80, D81, D82, D83, D84, D85, D9, F1, J1, J2, MX1, MX10, MX11, MX12, MX13, MX14, MX15, MX16, MX17, MX18, MX19, MX2, MX20, MX21, MX22, MX23, MX24, MX25, MX26, MX27, MX28, MX29, MX3, MX30, MX31, MX32, MX33, MX34, MX35, MX36, MX37, MX38, MX39, MX4, MX40, MX41, MX42, MX43, MX44, MX45, MX46, MX47, MX48, MX49, MX5, MX50, MX51, MX52, MX53, MX54, MX55, MX56, MX57, MX58, MX59, MX6, MX60, MX61, MX62, MX63, MX64, MX65, MX66, MX67, MX68, MX69, MX7, MX70, MX71, MX72, MX73, MX74, MX75, MX76, MX77, MX78, MX79, MX8, MX80, MX81, MX82, MX83, MX84, MX9, R1, R11, R12, R2, R3, R4, R5, R6, R7, R8, R9, S1, S2, S3, S4, SW1, SW2, SW3, U1, U2, U3, U4, Y1: moved to B.Cu
- moved SW3 579.6 mm to (366.9, 50.3), turned to 90 degrees
- moved R12 555.5 mm to (365.5, 53.3), turned to -90 degrees
- moved R11 553.2 mm to (363.5, 53.3), turned to -90 degrees
- moved S2 551.5 mm to (333.4, 105.0)
- moved S3 546.7 mm to (335.8, 66.9)
- moved D84 504.8 mm to (356.4, 145.0), turned to 90 degrees
- moved D60 497.8 mm to (364.2, 108.9), turned to 0 degrees
- moved D74 497.2 mm to (356.2, 125.6), turned to 90 degrees
- moved D46 492.0 mm to (364.3, 89.8), turned to 0 degrees
- moved D83 485.3 mm to (337.2, 144.6), turned to 90 degrees
- moved D31 480.3 mm to (364.3, 70.7), turned to 0 degrees
- moved D73 477.8 mm to (337.0, 125.6), turned to 90 degrees
- moved D45 468.2 mm to (340.5, 89.7), turned to 0 degrees
- moved D59 466.9 mm to (333.4, 109.0), turned to 0 degrees
- moved D82 466.0 mm to (318.2, 144.6), turned to 90 degrees
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Routing:
- net +3V3: track 0.00 -> 313.8 mm, vias 0 -> 5
- net D+: track 0.00 -> 182.5 mm
- net D-: track 0.00 -> 180.9 mm
- net GND: track 0.00 -> 134.6 mm, vias 0 -> 20
- net Q_SEL: track 0.00 -> 46.4 mm
- net +1V1: track 0.00 -> 32.5 mm, vias 0 -> 2
- net RESET: track 0.00 -> 27.6 mm
- net Q_IO1: track 0.00 -> 24.5 mm
- net Q_IO2: track 0.00 -> 23.2 mm
- net VBUS: track 0.00 -> 17.0 mm
- net SWD: track 0.00 -> 13.9 mm
- net Q_IO3: track 0.00 -> 12.6 mm
- net Q_CLK: track 0.00 -> 12.2 mm
- net XIN: track 0.00 -> 12.2 mm
- net Q_IO0: track 0.00 -> 12.1 mm
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- added copper zone on B.Cu, net GND
- added copper zone on F.Cu, net GND
Other:
- board outline added: 305.4 x 132.6 mm
