File: KiCad/ze-keyboard.kicad_pcb (KiCad board)
At the start: 2 copper layers, 305.4 x 132.6 mm, 211 parts, among them J1 Conn_01x05, J2 USB_C_Receptacle_USB2.0, SW1 Flash, SW2 Reset, SW3 RotaryEncoder_Switch, U1 XC6206PxxxMR, U2 RP2040, U3 W25Q128JVS, U4 SRV05-4, Y1 Crystal_GND24_Small

Commit message: do some more stuff like fixing most of 90 degree traces
Routing:
- net Net-(D61-A): track 14.1 -> 5.37 mm
- net Net-(D64-A): track 14.0 -> 10.9 mm
- net Net-(D84-A): track 12.7 -> 9.60 mm
- net Net-(D75-A): track 13.0 -> 9.98 mm
- net Net-(D78-A): track 7.59 -> 4.59 mm
- net Net-(D77-A): track 13.0 -> 10.0 mm
- net Net-(D76-A): track 13.7 -> 10.7 mm
- net Net-(D80-A): track 12.9 -> 9.92 mm
- net Net-(D81-A): track 12.4 -> 9.46 mm
- net row4: track 472.1 -> 474.9 mm
- net Net-(D74-A): track 12.8 -> 9.95 mm
- net Net-(D63-A): track 13.2 -> 10.4 mm
- net Net-(D83-A): track 12.2 -> 9.50 mm
- net Net-(D79-A): track 13.0 -> 10.3 mm
- net Net-(D82-A): track 12.2 -> 9.49 mm
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