File: KiCad/ze-keyboard.kicad_pcb (KiCad board)
At the start: 2 copper layers, 305.4 x 132.6 mm, 211 parts, among them J1 Conn_01x05, J2 USB_C_Receptacle_USB2.0, SW1 Flash, SW2 Reset, SW3 RotaryEncoder_Switch, U1 XC6206PxxxMR, U2 RP2040, U3 W25Q128JVS, U4 SRV05-4, Y1 Crystal_GND24_Small

Commit message: stuff
Parts:
- turned S1 to 180 degrees
- turned S2 to 180 degrees
- turned S3 to 180 degrees
Routing:
- net row3: track 583.8 -> 584.9 mm
- net row1: track 668.7 -> 669.8 mm
- net row4: track 474.9 -> 475.7 mm
